File: swd-breakout.kicad_pcb (KiCad board)
At the start: 2 copper layers, 27.5 x 28 mm, 5 parts, among them J1 Conn_02x05_Odd_Even, J2 Conn_01x05_Socket, J3 Conn_01x05_Socket

Commit message: Updates
Parts:
- H1: footprint MountingHole:MountingHole_3.2mm_M3_ISO7380_Pad_TopBottom -> MountingHole:MountingHole_3.2mm_M3_ISO7380_Pad
Connections:
- H1 pad 1: (no net) -> unconnected-(H1-Pad1)
- H2 pad 1: (no net) -> unconnected-(H2-Pad1)_2
Changed lines of the file:
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@@
 	(net 9 "Net-(J1-Pin_10)")
 	(net 10 "Net-(J1-Pin_4)")
-	(footprint "MountingHole:MountingHole_3.2mm_M3_ISO7380_Pad_TopBottom"
+	(net 11 "unconnected-(H1-Pad1)")
+	(net 12 "unconnected-(H2-Pad1)")
+	(net 13 "unconnected-(H2-Pad1)_1")
+	(net 14 "unconnected-(H2-Pad1)_2")
+	(footprint "MountingHole:MountingHole_3.2mm_M3_ISO7380_Pad"
 		(layer "F.Cu")
 		(at 219 152)
@@
 			(at 0 -3.85 0)
 			(layer "F.SilkS")
-			(hide yes)
 			(effects
 				(font
@@
 			)
 		)
-		(property "Footprint" "MountingHole:MountingHole_3.2mm_M3_ISO7380_Pad_TopBottom"
+		(property "Footprint" "MountingHole:MountingHole_3.2mm_M3_ISO7380_Pad"
 			(at 0 0 0)
 			(unlocked yes)
@@
 			)
 		)
-		(property "Description" "Mounting Hole without connection"
+		(property "Description" "Mounting Hole with connection"
 			(at 0 0 0)
 			(unlocked yes)
@@
 			)
 		)
-		(property ki_fp_filters "MountingHole*")
+		(property ki_fp_filters "MountingHole*Pad*")
 		(sheetname "Root")
 		(sheetfile "swd-breakout.kicad_sch")
@@
 			(layer "F.CrtYd")
 		)
+		(fp_text user "${REFERENCE}"
+			(at 0 0 0)
+			(layer "F.Fab")
+			(effects
+				(font
+					(size 1 1)
+					(thickness 0.15)
+				)
+			)
+		)
 		(pad "1" thru_hole circle
 			(at 0 0)
-			(size 3.6 3.6)
+			(size 5.7 5.7)
 			(drill 3.2)
 			(layers "*.Cu" "*.Mask")
 			(remove_unused_layers no)
-		)
-		(pad "1" connect circle
-			(at 0 0)
-			(size 5.7 5.7)
-			(layers "F.Cu" "F.Mask")
-		)
-		(pad "1" connect circle
-			(at 0 0)
-			(size 5.7 5.7)
-			(layers "B.Cu" "B.Mask")
+			(net 11 "unconnected-(H1-Pad1)")
+			(pinfunction "1")
+			(pintype "input+no_connect")
 		)
 	)
@@
 			)
 		)
-		(property "Description" "Mounting Hole without connection"
+		(property "Description" "Mounting Hole with connection"
 			(at 0 0 0)
 			(unlocked yes)
@@
 			)
 		)
-		(property ki_fp_filters "MountingHole*")
+		(property ki_fp_filters "MountingHole*Pad*")
 		(sheetname "Root")
 		(sheetfile "swd-breakout.kicad_sch")
@@
 			(layers "*.Cu" "*.Mask")
 			(remove_unused_layers no)
+			(net 12 "unconnected-(H2-Pad1)")
+			(pinfunction "1")
+			(pintype "input+no_connect")
 		)
 		(pad "1" connect circle
@@
 			(size 5.7 5.7)
 			(layers "F.Cu" "F.Mask")
+			(net 13 "unconnected-(H2-Pad1)_1")
+			(pinfunction "1")
+			(pintype "input+no_connect")
 		)
 		(pad "1" connect circle
@@
 			(size 5.7 5.7)
 			(layers "B.Cu" "B.Mask")
+			(net 14 "unconnected-(H2-Pad1)_2")
+			(pinfunction "1")
+			(pintype "input+no_connect")
 		)
 	)
