File: swd-breakout.kicad_pcb (KiCad board)
At the start: 2 copper layers, 27.5 x 28 mm, 5 parts, among them J1 Conn_02x05_Odd_Even, J2 Conn_01x05_Socket, J3 Conn_01x05_Socket

Commit message: Connecting ground plane to GND pin via net
Connections:
- net Net-(J1-Pin_1) renamed /Vref
- net Net-(J1-Pin_10) renamed /~{RST}
- net Net-(J1-Pin_2) renamed /SWIO
- net Net-(J1-Pin_4) renamed /CLK
- net Net-(J1-Pin_6) renamed /SWO
- net Net-(J1-Pin_7) renamed /Key
- net Net-(J1-Pin_8) renamed /n/c
- J1 pad 3: Net-(J1-Pin_3) -> /GND
- J1 pad 5: Net-(J1-Pin_5) -> /GND
- J1 pad 9: Net-(J1-Pin_9) -> /GND
- J2 pad 2: Net-(J1-Pin_3) -> /GND
- J2 pad 3: Net-(J1-Pin_5) -> /GND
- J2 pad 5: Net-(J1-Pin_9) -> /GND
Routing:
- net /GND: track 0.00 -> 18.2 mm
- net Net-(J1-Pin_9): track 6.58 -> 0.00 mm
- net Net-(J1-Pin_3): track 6.08 -> 0.00 mm
- net Net-(J1-Pin_5): track 5.55 -> 0.00 mm
- added copper zone on B.Cu, net /GND
- removed copper zone on B.Cu, net (none)
